File: KiCad/ActiveLoad.sch (KiCad schematic (older format))
At the start: 63 parts, among them J1 AuxPower, J2 TWI, J3 PDI, J4 TC74X-3.3, J5 PowerInput, J6 FAN, Q1 BC807, Q2 BC817, Q3 BD911, Q4 BD136, SW1 SW_SPDT, U1 LM78L33, U2 L78M12, U3 ATXMEGA32E5-AU, U4 LM358, U5 TL081

Commit message: PCB
Parts:
- removed C1: 47u, Capacitors_SMD:CP_Elec_6.3x5.8, symbol CP
- removed Q1: BC807, TO_SOT_Packages_SMD:SOT-23, symbol BC807
- removed R3: 13, Resistors_SMD:R_0805, symbol R
- removed U1: LM78L33, TO_SOT_Packages_SMD:SOT-89-3, symbol LM78L05_TO92
- added D1: 1N4148, Diodes_SMD:D_1206, symbol D
- added U1: UA78M33, TO_SOT_Packages_SMD:TO-252-2, symbol L7812
- gave numbers to parts that had none: 1
Connections:
- net +12V: now also SW2.1 (A); no longer SW2.2 (B)
- net +3V3: now also U4.8 (V+), U1.3 (OUT); no longer U4.8 (V+)
- net CURRENT_LEVEL: now also U3.29 (AC0OUT/AC7/ADC7/PA7)
- net DRAIN_CONTROL: now also U3.3 (DAC1/AC3/ADC3/PA3); no longer U3.4 (DAC0/AC2/ADC2/PA2)
- net ENC_A: now also U3.11 (IN2/SCK/XCK0/OC5B/OC4CHS/OC4B/PC5)
- net ENC_B: now also U3.12 (EXTCLK/OUT0/IN1/~SS~/OC5A/~OC4CLS~/OC4A/PC4)
- net ENC_Switch: now also U3.9 (AC0OUT/IN3/MOSI/TXD0/OC4DHS/OC4D/PC7)
- net FAN_CONTROL: now also U3.4 (DAC0/AC2/ADC2/PA2); no longer U3.3 (DAC1/AC3/ADC3/PA3)
- net GND: now also ROT1.1 (SW1), U4.4 (V-), D1.2 (A), U1.2 (GND); no longer ROT1.5 (SW2), U4.4 (V-)
- net VOLTAGE_LEVEL: now also U3.30 (AC1OUT/AC6/ADC6/PA6)
- net at U4.5 (+): now also R12.2; no longer R17.2
- net at R13.2, R14.2: now also U4.2 (-); no longer U4.6 (-)
- net at R12.1, R13.1: now also U4.1; no longer U4.7
- net at R16.2: now also U4.7; no longer U4.1
- net at C14.1, R11.2: now also U4.6 (-); no longer U4.2 (-)
- net at U4.3 (+): now also R17.2; no longer R12.2
- net at C18.1, J6.2 (Pin_2), Q4.2 (C)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: now also D1.1 (K)
- net at R5.1, R6.1: now also ROT1.5 (SW2); no longer ROT1.1 (SW1)
- net at C4.1, SW1.2 (B), U2.1 (IN): now also SW2.2 (B), U1.1 (IN); no longer SW2.3 (C)
Other:
- note added: "32E5 (1.2mA)\nDisplay 0111 100 (80mW, 25mA)\nTC74 1001 xxx (0.3mA)\nRot (1mA)\nLM358 (2mA)\n1. NC\n2. SDA\n3. GND\n4. SCK\n5. VDD"
- note removed: "Display 0111 100\nTC74 1001 xxx\n1. NC\n2. SDA\n3. GND\n4. SCK\n5. VDD"
- moved on the sheet: C18, C2, C3, C4, C7, C8, C9, R22, R5, R6, SW2, U2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
