File: KiCad/ActiveLoad.kicad_pcb (KiCad board)
At the start: 2 copper layers, 85.7 x 70 mm, 69 parts, among them J1 AuxPower, J2 OLED I2C, J3 PDI, J4 TC74X-3.3, J5 PowerInput, J6 FAN, Q2 BC817, Q3 BD911, Q4 BD136, SW1 SW_SPDT, SW2 SW_SPDT, U1 UA78M33, U2 L78M12, U3 ATXMEGA32E5-AU, U4 LM358, U5 TL081

Commit message: Brand new version
Parts:
- removed the REF** at (119.4, 52.7)
- removed the REF** at (119.4, 82.5)
- added D4: LED, Diodes_SMD:D_0805, B.Cu at (69.2, 98.4)
- added R3: 3k3, Resistors_SMD:R_0805, B.Cu at (72.4, 101.0)
- added REF**: MountingHole_7.5mm, Mounting_Holes:MountingHole_6mm, F.Cu at (119.4, 82.5)
- added REF**: MountingHole_7.5mm, Mounting_Holes:MountingHole_6mm, F.Cu at (119.4, 52.1)
- Q4: value BD136 -> BD140
- R11, R15: value 14k7 -> 15k42
- R13: value 3k -> 3k3
- R21: value 510 -> 680
- U4: value LM358 -> OPA2170
- U5: value TL081 -> LM7321
- moved R24 12.5 mm to (67.3, 54.0), turned to 0 degrees
- moved R22 7.85 mm to (96.5, 65.4), turned to 0 degrees
- moved R25 7.75 mm to (64.1, 54.6), turned to 90 degrees
- moved R26 6.75 mm to (90.8, 58.4), turned to 90 degrees
- moved C7 5.39 mm to (97.2, 72.4)
- moved R6 4.62 mm to (100.3, 77.5)
- moved R5 4.02 mm to (99.1, 74.9), turned to 180 degrees
- moved R21 3.86 mm to (83.2, 62.2), turned to 0 degrees
- moved C17 3.59 mm to (88.3, 68.6), turned to 180 degrees
- moved R2 2.69 mm to (66.7, 64.1)
- moved J2 2.29 mm to (69.2, 65.4)
- moved R17 2.01 mm to (78.7, 62.2), turned to 0 degrees
- moved R1 1.80 mm to (74.3, 68.6)
- moved R7 1.80 mm to (101.0, 81.9), turned to 0 degrees
- moved R15 1.42 mm to (95.9, 61.6), turned to 180 degrees
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Connections:
- C15 pad 2: +3V3 -> +12V
- J6 pad 1: GND -> Net-(J6-Pad1)
- J6 pad 3: Net-(J6-Pad3) -> GND
- R21 pad 1: PowerInput -> Net-(Q2-Pad3)
- R21 pad 2: Net-(Q2-Pad3) -> +12V
- ROT1 pad 1: GND -> Net-(R5-Pad1)
- ROT1 pad 5: Net-(R5-Pad1) -> GND
- U3 pad 25: Net-(U3-Pad25) -> LED
- U4 pad 8: +3V3 -> +12V
Routing:
- net +12V: track 67.7 -> 88.3 mm, vias 2 -> 3
- net PowerInput: track 94.8 -> 75.7 mm
- net VOLTAGE_LEVEL: track 57.5 -> 67.3 mm
- net LED: track 0.00 -> 7.05 mm
- net +3V3: track 171.3 -> 165.1 mm, vias 5 -> 4
- net GND: track 373.4 -> 367.6 mm
- net Net-(Q4-Pad3): track 12.1 -> 7.12 mm
- net Net-(R19-Pad2): track 9.92 -> 5.51 mm
- net FAN_CONTROL: track 38.0 -> 42.2 mm
- net Net-(C18-Pad1): track 39.7 -> 35.6 mm
- net Net-(D4-Pad1): track 0.00 -> 2.78 mm
- net ENC_A: track 20.6 -> 18.6 mm
- net ENC_Switch: track 30.4 -> 32.2 mm
- net Net-(C16-Pad1): track 7.62 -> 5.91 mm
- net ENC_B: track 24.8 -> 23.3 mm
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Other:
- board text added: "ActiveLoad v2 2018.05.13, JP"
- board text added: "Aux Power 12V"
- board text added: "Input Power Max 25/35V"
- board text removed: "ActiveLoad v1 2018.04.05, JP"
- board text removed: "Aux Power"
- board text removed: "Input Power"
