File: KiCad/ActiveLoadMosfets/ActiveLoadMosfets.sch (KiCad schematic (older format))
At the start: 30 parts, among them J1 Conn_01x02_Male, Q1 STP60NF06L, Q2 STP60NF06L, Q3 STP60NF06L, Q4 STP60NF06L, Q5 STP60NF06L, Q6 STP60NF06L, U1 LM7322, U2 LM78M12

Commit message: PCB init
Parts:
- C1, C2, C3, C4, C5: footprint (none) -> Capacitors_SMD:C_0805
- C6: footprint (none) -> Capacitors_SMD:CP_Elec_4x5.8
- J1: footprint (none) -> Connectors_Terminal_Blocks:TerminalBlock_Altech_AK300-2_P5.00mm
- Q1, Q2, Q3, Q4, Q5, Q6: footprint (none) -> TO_SOT_Packages_THT:TO-220-3_Horizontal
- R1, R10, R11, R12, R13, R2, R3, R4, R5, R6, R7, R9: footprint (none) -> Resistors_SMD:R_0805
- R8: footprint (none) -> JPResistors:R_Axial_Power_L48.0mm_W12.5mm_P50.8mm
- RV1, RV2: footprint (none) -> Pin_Headers:Pin_Header_Straight_1x03_Pitch2.54mm
- U1: footprint (none) -> Housings_SOIC:SOIC-8_3.9x4.9mm_Pitch1.27mm
- U2: footprint Package_TO_SOT_THT:TO-220-3_Vertical -> TO_SOT_Packages_SMD:TO-252-2_Rectifier
Changed lines of the file:
@@
 EESchema Schematic File Version 4
+LIBS:ActiveLoadMosfets-cache
 EELAYER 26 0
 EELAYER END
@@
 F 0 "Q1" H 5805 2996 50  0000 L CNN
 F 1 "STP60NF06L" H 5805 2905 50  0000 L CNN
-F 2 "" H 5800 3050 50  0001 C CNN
+F 2 "TO_SOT_Packages_THT:TO-220-3_Horizontal" H 5800 3050 50  0001 C CNN
 F 3 "~" H 5600 2950 50  0001 C CNN
 	1    5600 2950
@@
 F 0 "R7" H 5420 2796 50  0000 L CNN
 F 1 "51" H 5420 2705 50  0000 L CNN
-F 2 "" V 5280 2750 50  0001 C CNN
+F 2 "Resistors_SMD:R_0805" V 5280 2750 50  0001 C CNN
 F 3 "~" H 5350 2750 50  0001 C CNN
 	1    5350 2750
@@
 F 0 "Q2" H 6705 2996 50  0000 L CNN
 F 1 "STP60NF06L" H 6705 2905 50  0000 L CNN
-F 2 "" H 6700 3050 50  0001 C CNN
+F 2 "TO_SOT_Packages_THT:TO-220-3_Horizontal" H 6700 3050 50  0001 C CNN
 F 3 "~" H 6500 2950 50  0001 C CNN
 	1    6500 2950
@@
 F 0 "R9" H 6320 2796 50  0000 L CNN
 F 1 "51" H 6320 2705 50  0000 L CNN
-F 2 "" V 6180 2750 50  0001 C CNN
+F 2 "Resistors_SMD:R_0805" V 6180 2750 50  0001 C CNN
 F 3 "~" H 6250 2750 50  0001 C CNN
 	1    6250 2750
@@
 F 0 "Q3" H 7605 2996 50  0000 L CNN
 F 1 "STP60NF06L" H 7605 2905 50  0000 L CNN
-F 2 "" H 7600 3050 50  0001 C CNN
+F 2 "TO_SOT_Packages_THT:TO-220-3_Horizontal" H 7600 3050 50  0001 C CNN
 F 3 "~" H 7400 2950 50  0001 C CNN
 	1    7400 2950
@@
 F 0 "R10" H 7220 2796 50  0000 L CNN
 F 1 "51" H 7220 2705 50  0000 L CNN
-F 2 "" V 7080 2750 50  0001 C CNN
+F 2 "Resistors_SMD:R_0805" V 7080 2750 50  0001 C CNN
 F 3 "~" H 7150 2750 50  0001 C CNN
 	1    7150 2750
@@
 F 0 "Q4" H 8505 2996 50  0000 L CNN
 F 1 "STP60NF06L" H 8505 2905 50  0000 L CNN
-F 2 "" H 8500 3050 50  0001 C CNN
+F 2 "TO_SOT_Packages_THT:TO-220-3_Horizontal" H 8500 3050 50  0001 C CNN
 F 3 "~" H 8300 2950 50  0001 C CNN
 	1    8300 2950
@@
 F 0 "R11" H 8120 2796 50  0000 L CNN
 F 1 "51" H 8120 2705 50  0000 L CNN
-F 2 "" V 7980 2750 50  0001 C CNN
+F 2 "Resistors_SMD:R_0805" V 7980 2750 50  0001 C CNN
 F 3 "~" H 8050 2750 50  0001 C CNN
 	1    8050 2750
@@
 F 0 "R8" H 5770 3596 50  0000 L CNN
 F 1 "0R1" H 5770 3505 50  0000 L CNN
-F 2 "" V 5630 3550 50  0001 C CNN
+F 2 "JPResistors:R_Axial_Power_L48.0mm_W12.5mm_P50.8mm" V 5630 3550 50  0001 C CNN
 F 3 "~" H 5700 3550 50  0001 C CNN
 	1    5700 3550
@@
 F 0 "Q5" H 9405 2996 50  0000 L CNN
 F 1 "STP60NF06L" H 9405 2905 50  0000 L CNN
-F 2 "" H 9400 3050 50  0001 C CNN
+F 2 "TO_SOT_Packages_THT:TO-220-3_Horizontal" H 9400 3050 50  0001 C CNN
 F 3 "~" H 9200 2950 50  0001 C CNN
 	1    9200 2950
@@
 F 0 "R12" H 9020 2796 50  0000 L CNN
 F 1 "51" H 9020 2705 50  0000 L CNN
-F 2 "" V 8880 2750 50  0001 C CNN
+F 2 "Resistors_SMD:R_0805" V 8880 2750 50  0001 C CNN
 F 3 "~" H 8950 2750 50  0001 C CNN
 	1    8950 2750
@@
 F 0 "Q6" H 10305 2996 50  0000 L CNN
 F 1 "STP60NF06L" H 10305 2905 50  0000 L CNN
-F 2 "" H 10300 3050 50  0001 C CNN
+F 2 "TO_SOT_Packages_THT:TO-220-3_Horizontal" H 10300 3050 50  0001 C CNN
 F 3 "~" H 10100 2950 50  0001 C CNN
 	1    10100 2950
@@
 F 0 "R13" H 9920 2796 50  0000 L CNN
 F 1 "51" H 9920 2705 50  0000 L CNN
-F 2 "" V 9780 2750 50  0001 C CNN
+F 2 "Resistors_SMD:R_0805" V 9780 2750 50  0001 C CNN
 F 3 "~" H 9850 2750 50  0001 C CNN
 	1    9850 2750
@@
 F 0 "R6" V 5043 3250 50  0000 C CNN
 F 1 "1k" V 5134 3250 50  0000 C CNN
-F 2 "" V 5180 3250 50  0001 C CNN
+F 2 "Resistors_SMD:R_0805" V 5180 3250 50  0001 C CNN
 F 3 "~" H 5250 3250 50  0001 C CNN
 	1    5250 3250
@@
 F 0 "U1" H 3550 2867 50  0000 C CNN
 F 1 "LM7322" H 3550 2776 50  0000 C CNN
-F 2 "" H 3550 2500 50  0001 C CNN
+F 2 "Housings_SOIC:SOIC-8_3.9x4.9mm_Pitch1.27mm" H 3550 2500 50  0001 C CNN
 F 3 "~" H 3550 2500 50  0001 C CNN
 	3    3550 2500
@@
 F 0 "U1" H 4350 3717 50  0000 C CNN
 F 1 "LM7322" H 4350 3626 50  0000 C CNN
-F 2 "" H 4350 3350 50  0001 C CNN
+F 2 "Housings_SOIC:SOIC-8_3.9x4.9mm_Pitch1.27mm" H 4350 3350 50  0001 C CNN
 F 3 "~" H 4350 3350 50  0001 C CNN
 	1    4350 3350
@@
 F 0 "R5" H 4680 3654 50  0000 R CNN
 F 1 "1k" H 4680 3745 50  0000 R CNN
-F 2 "" V 4680 3700 50  0001 C CNN
+F 2 "Resistors_SMD:R_0805" V 4680 3700 50  0001 C CNN
 F 3 "~" H 4750 3700 50  0001 C CNN
 	1    4750 3700
@@
 F 0 "J1" H 2756 1078 50  0000 C CNN
 F 1 "Conn_01x02_Male" H 2756 987 50  0000 C CNN
-F 2 "" H 2650 900 50  0001 C CNN
+F 2 "Connectors_Terminal_Blocks:TerminalBlock_Altech_AK300-2_P5.00mm" H 2650 900 50  0001 C CNN
 F 3 "~" H 2650 900 50  0001 C CNN
 	1    2650 900
@@
 F 0 "R4" V 4143 2850 50  0000 C CNN
 F 1 "5k" V 4234 2850 50  0000 C CNN
-F 2 "" V 4280 2850 50  0001 C CNN
+F 2 "Resistors_SMD:R_0805" V 4280 2850 50  0001 C CNN
 F 3 "~" H 4350 2850 50  0001 C CNN
 	1    4350 2850
@@
 F 0 "R3" H 3130 2904 50  0000 R CNN
 F 1 "10k" H 3130 2995 50  0000 R CNN
-F 2 "" V 3130 2950 50  0001 C CNN
+F 2 "Resistors_SMD:R_0805" V 3130 2950 50  0001 C CNN
 F 3 "~" H 3200 2950 50  0001 C CNN
 	1    3200 2950
@@
 F 0 "C5" H 4865 2746 50  0000 L CNN
 F 1 "3n3" H 4865 2655 50  0000 L CNN
-F 2 "" H 4788 2550 50  0001 C CNN
+F 2 "Capacitors_SMD:C_0805" H 4788 2550 50  0001 C CNN
 F 3 "~" H 4750 2700 50  0001 C CNN
 	1    4750 2700
@@
 F 0 "R2" V 2343 2400 50  0000 C CNN
 F 1 "5k" V 2434 2400 50  0000 C CNN
-F 2 "" V 2480 2400 50  0001 C CNN
+F 2 "Resistors_SMD:R_0805" V 2480 2400 50  0001 C CNN
 F 3 "~" H 2550 2400 50  0001 C CNN
 	1    2550 2400
@@
 F 0 "C1" H 2965 2696 50  0000 L CNN
 F 1 "220n" H 2965 2605 50  0000 L CNN
-F 2 "" H 2888 2500 50  0001 C CNN
+F 2 "Capacitors_SMD:C_0805" H 2888 2500 50  0001 C CNN
 F 3 "~" H 2850 2650 50  0001 C CNN
 	1    2850 2650
@@
 F 0 "RV1" H 2030 2446 50  0000 R CNN
 F 1 "47k" H 2030 2355 50  0000 R CNN
-F 2 "" H 2100 2400 50  0001 C CNN
+F 2 "Pin_Headers:Pin_Header_Straight_1x03_Pitch2.54mm" H 2100 2400 50  0001 C CNN
 F 3 "~" H 2100 2400 50  0001 C CNN
 	1    2100 2400
@@
 F 0 "RV2" H 2030 2846 50  0000 R CNN
 F 1 "1k" H 2030 2755 50  0000 R CNN
-F 2 "" H 2100 2800 50  0001 C CNN
+F 2 "Pin_Headers:Pin_Header_Straight_1x03_Pitch2.54mm" H 2100 2800 50  0001 C CNN
 F 3 "~" H 2100 2800 50  0001 C CNN
 	1    2100 2800
@@
 F 0 "R1" H 2030 1954 50  0000 R CNN
 F 1 "47k" H 2030 2045 50  0000 R CNN
-F 2 "" V 2030 2000 50  0001 C CNN
+F 2 "Resistors_SMD:R_0805" V 2030 2000 50  0001 C CNN
 F 3 "~" H 2100 2000 50  0001 C CNN
 	1    2100 2000
@@
 F 0 "C3" V 3748 2100 50  0000 C CNN
 F 1 "100n" V 3839 2100 50  0000 C CNN
-F 2 "" H 4038 1950 50  0001 C CNN
+F 2 "Capacitors_SMD:C_0805" H 4038 1950 50  0001 C CNN
 F 3 "~" H 4000 2100 50  0001 C CNN
 	1    4000 2100
@@
 F 0 "U2" H 4350 1142 50  0000 C CNN
 F 1 "LM78M12" H 4350 1051 50  0000 C CNN
-F 2 "Package_TO_SOT_THT:TO-220-3_Vertical" H 4350 1125 50  0001 C CIN
+F 2 "TO_SOT_Packages_SMD:TO-252-2_Rectifier" H 4350 1125 50  0001 C CIN
 F 3 "http://www.fairchildsemi.com/ds/LM/LM7805.pdf" H 4350 850 50  0001 C CNN
 	1    4350 900
@@
 F 0 "C4" H 4865 1196 50  0000 L CNN
 F 1 "100n" H 4865 1105 50  0000 L CNN
-F 2 "" H 4788 1000 50  0001 C CNN
+F 2 "Capacitors_SMD:C_0805" H 4788 1000 50  0001 C CNN
 F 3 "~" H 4750 1150 50  0001 C CNN
 	1    4750 1150
@@
 F 0 "C2" H 4065 1196 50  0000 L CNN
 F 1 "470n" H 4065 1105 50  0000 L CNN
-F 2 "" H 3988 1000 50  0001 C CNN
+F 2 "Capacitors_SMD:C_0805" H 3988 1000 50  0001 C CNN
 F 3 "~" H 3950 1150 50  0001 C CNN
 	1    3950 1150
@@
 F 0 "C6" H 5268 1196 50  0000 L CNN
 F 1 "10u" H 5268 1105 50  0000 L CNN
-F 2 "" H 5188 1000 50  0001 C CNN
+F 2 "Capacitors_SMD:CP_Elec_4x5.8" H 5188 1000 50  0001 C CNN
 F 3 "~" H 5150 1150 50  0001 C CNN
 	1    5150 1150
@@
 F 0 "U1" H 3708 2546 50  0000 L CNN
 F 1 "LM7322" H 3708 2455 50  0000 L CNN
-F 2 "" H 3750 2500 50  0001 C CNN
+F 2 "Housings_SOIC:SOIC-8_3.9x4.9mm_Pitch1.27mm" H 3750 2500 50  0001 C CNN
 F 3 "~" H 3750 2500 50  0001 C CNN
 	2    3750 2500

Commit message: pcb work
Parts:
- added C10, C12: 10u, Capacitors_SMD:CP_Elec_4x5.8, symbol Device:CP
- added C11, C13, C15, C16, C8: 100n, Capacitors_SMD:C_0805, symbol Device:C
- added C14, C19: 10n, Capacitors_SMD:C_0805, symbol Device:C
- added C17, C18: 1u, Capacitors_SMD:C_0805, symbol Device:C
- added C7, C9: 47u, Capacitors_SMD:CP_Elec_6.3x5.8, symbol Device:CP
- added J2: Conn_02x03_Odd_Even, Pin_Headers:Pin_Header_Straight_2x03_Pitch2.54mm, symbol Connector_Generic:Conn_02x03_Odd_Even
- added L1: 10u, Inductors_SMD:L_0805, symbol Device:L
- added Q7, Q8, Q9: IRLML2244, TO_SOT_Packages_SMD:SOT-23, symbol Transistor_FET:IRLML6402
- added R14: 10k, Resistors_SMD:R_0805, symbol Device:R
- added R15, R16, R17, R19: 1k, Resistors_SMD:R_0805, symbol Device:R
- added R18, R20: 10, Resistors_SMD:R_1206, symbol Device:R
- added U3: ATxmega32E5-AU, Housings_QFP:TQFP-32_7x7mm_Pitch0.8mm, symbol MCU_Microchip_ATmega:ATxmega32E5-AU
- added U4, U8: LED-3digits, JPDisplays:LED-14.2x3, symbol myLib:LED-3digits
- added U5: LM78M33, TO_SOT_Packages_SMD:TO-252-2_Rectifier, symbol Regulator_Linear:LM7812_TO220
- added U6, U7: SCT2167, Housings_SOIC:SOIC-16_3.9x9.9mm_Pitch1.27mm, symbol myLib:SCT2167
- C6: value 10u -> 47u; footprint Capacitors_SMD:CP_Elec_4x5.8 -> Capacitors_SMD:CP_Elec_6.3x5.8
- RV1, RV2: footprint Pin_Headers:Pin_Header_Straight_1x03_Pitch2.54mm -> Connectors_Terminal_Blocks:TerminalBlock_bornier-3_P5.08mm
Connections:
- net labels added: +3.3V, +3.3Va, CURRENT, Digit1, Digit2, Digit3, Latch, MOSI, OutputEnabled, PDI_CLK, PDI_DATA, SCK, VOLTAGE
- wire segments 88 -> 218
- no-connect marks 1 -> 21
Other:
- moved on the sheet: C1, C2, C3, C4, C5, C6, J1, Q1, Q2, Q3, Q4, Q5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

Commit message: More pcb work
Parts:
- removed C10: 10u, Capacitors_SMD:CP_Elec_4x5.8, symbol Device:CP
- added C10: 100n, Capacitors_SMD:C_0805, symbol Device:C
- added C20: 10n, Capacitors_SMD:C_0805, symbol Device:C
- added D1: LED, LEDs:LED_0805, symbol Device:LED
- added R21, R22, R23: 10k, Resistors_SMD:R_0805, symbol Device:R
- added SW1: SW_SPST, Buttons_Switches_SMD:SW_SPST_B3SL-1002P, symbol Switch:SW_SPST
Connections:
- net labels added: LED, SWITCH
- wire segments 218 -> 223
Other:
- moved on the sheet: C8, C9, U5

Commit message: PCB Proofed
Parts:
- added SW2: SW_SPDT, JPConnectors:SlideSwitch3Poles, symbol Switch:SW_SPDT
- RV1, RV2: footprint Connectors_Terminal_Blocks:TerminalBlock_bornier-3_P5.08mm -> JPResistors:Pot_PCB-mount
- SW1: footprint Buttons_Switches_SMD:SW_SPST_B3SL-1002P -> Buttons_Switches_SMD:SW_SPST_B3S-1000
Connections:
- wire segments 223 -> 226
- no-connect marks 21 -> 19
Other:
- moved on the sheet: C10, C8, C9, U5
Changed lines of the file:
@@
 F 0 "RV1" H 1780 1296 50  0000 R CNN
 F 1 "47k" H 1780 1205 50  0000 R CNN
-F 2 "Connectors_Terminal_Blocks:TerminalBlock_bornier-3_P5.08mm" H 1850 1250 50  0001 C CNN
+F 2 "JPResistors:Pot_PCB-mount" H 1850 1250 50  0001 C CNN
 F 3 "~" H 1850 1250 50  0001 C CNN
 	1    1850 1250
-	1    0    0    -1
+	1    0    0    1
 $EndComp
 $Comp
@@
 F 0 "RV2" H 1780 1696 50  0000 R CNN
 F 1 "1k" H 1780 1605 50  0000 R CNN
-F 2 "Connectors_Terminal_Blocks:TerminalBlock_bornier-3_P5.08mm" H 1850 1650 50  0001 C CNN
+F 2 "JPResistors:Pot_PCB-mount" H 1850 1650 50  0001 C CNN
 F 3 "~" H 1850 1650 50  0001 C CNN
 	1    1850 1650
-	1    0    0    -1
+	1    0    0    1
 $EndComp
 $Comp
@@
 L Regulator_Linear:LM7812_TO220 U5
 U 1 1 5B8E3591
-P 3150 3200
-F 0 "U5" H 3150 3442 50  0000 C CNN
-F 1 "LM78M33" H 3150 3351 50  0000 C CNN
-F 2 "TO_SOT_Packages_SMD:TO-252-2_Rectifier" H 3150 3425 50  0001 C CIN
-F 3 "http://www.fairchildsemi.com/ds/LM/LM7805.pdf" H 3150 3150 50  0001 C CNN
-	1    3150 3200
+P 3600 3300
+F 0 "U5" H 3600 3542 50  0000 C CNN
+F 1 "LM78M33" H 3600 3451 50  0000 C CNN
+F 2 "TO_SOT_Packages_SMD:TO-252-2_Rectifier" H 3600 3525 50  0001 C CIN
+F 3 "http://www.fairchildsemi.com/ds/LM/LM7805.pdf" H 3600 3250 50  0001 C CNN
+	1    3600 3300
 	1    0    0    -1
 $EndComp
@@
 L Device:C C8
 U 1 1 5B8E36F8
-P 2650 3450
-F 0 "C8" H 2765 3496 50  0000 L CNN
-F 1 "100n" H 2765 3405 50  0000 L CNN
-F 2 "Capacitors_SMD:C_0805" H 2688 3300 50  0001 C CNN
-F 3 "~" H 2650 3450 50  0001 C CNN
-	1    2650 3450
+P 3100 3550
+F 0 "C8" H 3215 3596 50  0000 L CNN
+F 1 "100n" H 3215 3505 50  0000 L CNN
+F 2 "Capacitors_SMD:C_0805" H 3138 3400 50  0001 C CNN
+F 3 "~" H 3100 3550 50  0001 C CNN
+	1    3100 3550
 	1    0    0    -1
 $EndComp
@@
 L Device:CP C9
 U 1 1 5B8EE733
-P 3850 3450
-F 0 "C9" H 3968 3496 50  0000 L CNN
-F 1 "47u" H 3968 3405 50  0000 L CNN
-F 2 "Capacitors_SMD:CP_Elec_6.3x5.8" H 3888 3300 50  0001 C CNN
-F 3 "~" H 3850 3450 50  0001 C CNN
-	1    3850 3450
-	1    0    0    -1
-$EndComp
-Wire Wire Line
-	3850 3200 3850 3300
+P 4300 3550
+F 0 "C9" H 4418 3596 50  0000 L CNN
+F 1 "47u" H 4418 3505 50  0000 L CNN
+F 2 "Capacitors_SMD:CP_Elec_6.3x5.8" H 4338 3400 50  0001 C CNN
+F 3 "~" H 4300 3550 50  0001 C CNN
+	1    4300 3550
+	1    0    0    -1
+$EndComp
+Wire Wire Line
+	4300 3300 4300 3400
 $Comp
 L power:GND #PWR0114
@@
 L power:GND #PWR0115
 U 1 1 5B8F43CC
-P 3150 3500
-F 0 "#PWR0115" H 3150 3250 50  0001 C CNN
-F 1 "GND" H 3155 3327 50  0000 C CNN
-F 2 "" H 3150 3500 50  0001 C CNN
-F 3 "" H 3150 3500 50  0001 C CNN
-	1    3150 3500
+P 3600 3600
+F 0 "#PWR0115" H 3600 3350 50  0001 C CNN
+F 1 "GND" H 3605 3427 50  0000 C CNN
+F 2 "" H 3600 3600 50  0001 C CNN
+F 3 "" H 3600 3600 50  0001 C CNN
+	1    3600 3600
 	1    0    0    -1
 $EndComp
@@
 L power:GND #PWR0116
 U 1 1 5B8F443D
-P 2650 3600
-F 0 "#PWR0116" H 2650 3350 50  0001 C CNN
-F 1 "GND" H 2655 3427 50  0000 C CNN
-F 2 "" H 2650 3600 50  0001 C CNN
-F 3 "" H 2650 3600 50  0001 C CNN
-	1    2650 3600
+P 3100 3700
+F 0 "#PWR0116" H 3100 3450 50  0001 C CNN
+F 1 "GND" H 3105 3527 50  0000 C CNN
+F 2 "" H 3100 3700 50  0001 C CNN
+F 3 "" H 3100 3700 50  0001 C CNN
+	1    3100 3700
 	1    0    0    -1
 $EndComp
@@
 L power:GND #PWR0117
 U 1 1 5B8F44AE
-P 3850 3600
-F 0 "#PWR0117" H 3850 3350 50  0001 C CNN
-F 1 "GND" H 3855 3427 50  0000 C CNN
-F 2 "" H 3850 3600 50  0001 C CNN
-F 3 "" H 3850 3600 50  0001 C CNN
-	1    3850 3600
+P 4300 3700
+F 0 "#PWR0117" H 4300 3450 50  0001 C CNN
+F 1 "GND" H 4305 3527 50  0000 C CNN
+F 2 "" H 4300 3700 50  0001 C CNN
+F 3 "" H 4300 3700 50  0001 C CNN
+	1    4300 3700
 	1    0    0    -1
 $EndComp
@@
 L power:+3.3V #PWR0118
 U 1 1 5B8F451F
-P 3850 3100
-F 0 "#PWR0118" H 3850 2950 50  0001 C CNN
-F 1 "+3.3V" H 3865 3273 50  0000 C CNN
-F 2 "" H 3850 3100 50  0001 C CNN
-F 3 "" H 3850 3100 50  0001 C CNN
-	1    3850 3100
-	1    0    0    -1
-$EndComp
-Wire Wire Line
-	3850 3100 3850 3200
-Connection ~ 3850 3200
+P 4300 3200
+F 0 "#PWR0118" H 4300 3050 50  0001 C CNN
+F 1 "+3.3V" H 4315 3373 50  0000 C CNN
+F 2 "" H 4300 3200 50  0001 C CNN
+F 3 "" H 4300 3200 50  0001 C CNN
+	1    4300 3200
+	1    0    0    -1
+$EndComp
+Wire Wire Line
+	4300 3200 4300 3300
+Connection ~ 4300 3300
 Wire Wire Line
 	800  3300 800  3200
 Connection ~ 800  3200
 Wire Wire Line
-	2850 3200 2650 3200
+	3300 3300 3100 3300
 $Comp
 L Device:R R18
@@
 NoConn ~ 4150 6800
 NoConn ~ 4150 6600
-NoConn ~ 4150 6500
-NoConn ~ 4150 6400
 NoConn ~ 4150 5600
 NoConn ~ 4150 5700
@@
 OutputEnabled
 Wire Wire Line
-	3450 3200 3550 3200
-Wire Wire Line
-	2650 3300 2650 3200
-Connection ~ 2650 3200
-Wire Wire Line
-	2650 3200 2350 3200
+	3900 3300 4000 3300
+Wire Wire Line
+	3100 3400 3100 3300
+Connection ~ 3100 3300
+Wire Wire Line
+	3100 3300 2800 3300
 $Comp
 L Device:C C10
 U 1 1 5BD47ED4
-P 3550 3450
-F 0 "C10" H 3665 3496 50  0000 L CNN
-F 1 "100n" H 3665 3405 50  0000 L CNN
-F 2 "Capacitors_SMD:C_0805" H 3588 3300 50  0001 C CNN
-F 3 "~" H 3550 3450 50  0001 C CNN
-	1    3550 3450
+P 4000 3550
+F 0 "C10" H 4115 3596 50  0000 L CNN
+F 1 "100n" H 4115 3505 50  0000 L CNN
+F 2 "Capacitors_SMD:C_0805" H 4038 3400 50  0001 C CNN
+F 3 "~" H 4000 3550 50  0001 C CNN
+	1    4000 3550
 	1    0    0    -1
 $EndComp
@@
 L power:GND #PWR0104
 U 1 1 5BD98B8C
-P 3550 3600
-F 0 "#PWR0104" H 3550 3350 50  0001 C CNN
-F 1 "GND" H 3555 3427 50  0000 C CNN
-F 2 "" H 3550 3600 50  0001 C CNN
-F 3 "" H 3550 3600 50  0001 C CNN
-	1    3550 3600
-	1    0    0    -1
-$EndComp
-Wire Wire Line
-	3550 3300 3550 3200
-Connection ~ 3550 3200
-Wire Wire Line
-	3550 3200 3850 3200
+P 4000 3700
+F 0 "#PWR0104" H 4000 3450 50  0001 C CNN
+F 1 "GND" H 4005 3527 50  0000 C CNN
+F 2 "" H 4000 3700 50  0001 C CNN
+F 3 "" H 4000 3700 50  0001 C CNN
+	1    4000 3700
+	1    0    0    -1
+$EndComp
+Wire Wire Line
+	4000 3400 4000 3300
+Connection ~ 4000 3300
+Wire Wire Line
+	4000 3300 4300 3300
 $Comp
 L Device:LED D1
@@
 F 0 "SW1" V 6254 4198 50  0000 L CNN
 F 1 "SW_SPST" V 6345 4198 50  0000 L CNN
-F 2 "Buttons_Switches_SMD:SW_SPST_B3SL-1002P" H 6300 4100 50  0001 C CNN
+F 2 "Buttons_Switches_SMD:SW_SPST_B3S-1000" H 6300 4100 50  0001 C CNN
 F 3 "" H 6300 4100 50  0001 C CNN
 	1    6300 4100
@@
 	2750 6500 2600 6500
 NoConn ~ 2750 6700
+Text GLabel 4350 6500 2    50   Input ~ 0
+SWITCH
+Text GLabel 4350 6400 2    50   Input ~ 0
+LED
+Wire Wire Line
+	4350 6400 4150 6400
+Wire Wire Line
+	4150 6500 4350 6500
+$Comp
+L Switch:SW_SPDT SW2
+U 1 1 5BE4E4C5
+P 2600 3200
+F 0 "SW2" H 2600 3485 50  0000 C CNN
+F 1 "SW_SPDT" H 2600 3394 50  0000 C CNN
+F 2 "JPConnectors:SlideSwitch3Poles" H 2600 3200 50  0001 C CNN
+F 3 "" H 2600 3200 50  0001 C CNN
+	1    2600 3200
+	1    0    0    -1
+$EndComp
+Wire Wire Line
+	2350 3200 2400 3200
 $EndSCHEMATC
