File: KiCad/ActiveLoadMosfets/ActiveLoadMosfets.sch (KiCad schematic (older format))
At the start: 68 parts, among them J1 Conn_01x02_Male, J2 Conn_02x03_Odd_Even, Q1 STP60NF06L, Q2 STP60NF06L, Q3 STP60NF06L, Q4 STP60NF06L, Q5 STP60NF06L, Q6 STP60NF06L, Q7 IRLML2244, Q8 IRLML2244, Q9 IRLML2244, SW1 SW_SPST, SW2 SW_SPDT, U1 TLV2372, U2 LM78M12, U3 ATxmega32E5-AU, U4 LED-3digits, U5 LM78M33, U6 SCT2167, U7 SCT2167, U8 LED-3digits

Commit message: More c++ code, bug fixes on the PCB
Parts:
- added C?: 10u, Capacitors_SMD:CP_Elec_4x5.8, symbol Device:CP
- added R?: 1k1, Resistors_SMD:R_0805, symbol Device:R
- C5: value 3n3 -> 1n
- R15, R19: value 1k -> 5k
- R16: value 1k -> 47k
- R17: value 1k -> 1k1
- R4: value 5k -> 5k / 47k ?
Connections:
- wire segments 226 -> 229
- no-connect marks 19 -> 20
Other:
- moved on the sheet: C5
Changed lines of the file:
@@
 	1    0    0    -1
 $EndComp
-Text Notes 5750 2750 0    50   ~ 0
+Text Notes 5550 2750 0    50   ~ 0
 Imax=10A\nUmax=1V
 Text Notes 4400 950  0    50   ~ 0
@@
 P 4100 1700
 F 0 "R4" V 3893 1700 50  0000 C CNN
-F 1 "5k" V 3984 1700 50  0000 C CNN
+F 1 "5k / 47k ?" V 3984 1700 50  0000 C CNN
 F 2 "Resistors_SMD:R_0805" V 4030 1700 50  0001 C CNN
 F 3 "~" H 4100 1700 50  0001 C CNN
@@
 Wire Wire Line
 	2950 2200 2950 1950
-Wire Wire Line
-	3800 1350 4500 1350
 Connection ~ 5100 1350
 $Comp
 L Device:C C5
 U 1 1 5B75BACA
-P 4500 1550
-F 0 "C5" H 4615 1596 50  0000 L CNN
-F 1 "3n3" H 4615 1505 50  0000 L CNN
-F 2 "Capacitors_SMD:C_0805" H 4538 1400 50  0001 C CNN
-F 3 "~" H 4500 1550 50  0001 C CNN
-	1    4500 1550
-	1    0    0    -1
-$EndComp
-Wire Wire Line
-	4500 1400 4500 1350
-Connection ~ 4500 1350
-Wire Wire Line
-	4500 1350 5100 1350
+P 4700 1500
+F 0 "C5" H 4815 1546 50  0000 L CNN
+F 1 "1n" H 4815 1455 50  0000 L CNN
+F 2 "Capacitors_SMD:C_0805" H 4738 1350 50  0001 C CNN
+F 3 "~" H 4700 1500 50  0001 C CNN
+	1    4700 1500
+	1    0    0    -1
+$EndComp
 $Comp
 L Device:R R2
@@
 Wire Wire Line
 	4500 1700 4500 2300
-Connection ~ 4500 1700
 Connection ~ 4500 2300
 $Comp
@@
 Wire Wire Line
 	2300 2400 2200 2400
+Text GLabel 1450 2600 0    50   Input ~ 0
+PDI_CLK
 Text GLabel 1450 2400 0    50   Input ~ 0
-PDI_CLK
-Text GLabel 1450 2600 0    50   Input ~ 0
 PDI_DATA
 Wire Wire Line
@@
 P 6300 6150
 F 0 "R15" H 6230 6104 50  0000 R CNN
-F 1 "1k" H 6230 6195 50  0000 R CNN
+F 1 "5k" H 6230 6195 50  0000 R CNN
 F 2 "Resistors_SMD:R_0805" V 6230 6150 50  0001 C CNN
 F 3 "~" H 6300 6150 50  0001 C CNN
@@
 Wire Wire Line
 	5200 2100 5450 2100
-Text GLabel 5600 2200 2    50   Input ~ 0
+Text GLabel 6200 2200 2    50   Input ~ 0
 CURRENT
 Wire Wire Line
@@
 P 7550 1050
 F 0 "R16" H 7480 1004 50  0000 R CNN
-F 1 "1k" H 7480 1095 50  0000 R CNN
+F 1 "47k" H 7480 1095 50  0000 R CNN
 F 2 "Resistors_SMD:R_0805" V 7480 1050 50  0001 C CNN
 F 3 "~" H 7550 1050 50  0001 C CNN
@@
 P 7950 1050
 F 0 "R17" H 7880 1004 50  0000 R CNN
-F 1 "1k" H 7880 1095 50  0000 R CNN
+F 1 "1k1" H 7880 1095 50  0000 R CNN
 F 2 "Resistors_SMD:R_0805" V 7880 1050 50  0001 C CNN
 F 3 "~" H 7950 1050 50  0001 C CNN
@@
 P 8900 6150
 F 0 "R19" H 8830 6104 50  0000 R CNN
-F 1 "1k" H 8830 6195 50  0000 R CNN
+F 1 "5k" H 8830 6195 50  0000 R CNN
 F 2 "Resistors_SMD:R_0805" V 8830 6150 50  0001 C CNN
 F 3 "~" H 8900 6150 50  0001 C CNN
@@
 Wire Wire Line
 	2350 3200 2400 3200
+Connection ~ 4700 1350
+Wire Wire Line
+	4700 1350 5100 1350
+Connection ~ 2950 1650
+Wire Wire Line
+	3800 1350 4700 1350
+Wire Wire Line
+	2950 1650 4700 1650
+$Comp
+L Device:R R?
+U 1 1 5B9E9754
+P 5750 2200
+F 0 "R?" V 5543 2200 50  0000 C CNN
+F 1 "1k1" V 5634 2200 50  0000 C CNN
+F 2 "Resistors_SMD:R_0805" V 5680 2200 50  0001 C CNN
+F 3 "~" H 5750 2200 50  0001 C CNN
+	1    5750 2200
+	0    1    1    0
+$EndComp
+$Comp
+L Device:CP C?
+U 1 1 5B9E9EC7
+P 6050 2400
+F 0 "C?" H 6168 2446 50  0000 L CNN
+F 1 "10u" H 6168 2355 50  0000 L CNN
+F 2 "Capacitors_SMD:CP_Elec_4x5.8" H 6088 2250 50  0001 C CNN
+F 3 "~" H 6050 2400 50  0001 C CNN
+	1    6050 2400
+	1    0    0    -1
+$EndComp
+NoConn ~ 5450 2800
+$Comp
+L power:GND #PWR?
+U 1 1 5BA11FCB
+P 6050 2550
+F 0 "#PWR?" H 6050 2300 50  0001 C CNN
+F 1 "GND" H 6055 2377 50  0000 C CNN
+F 2 "" H 6050 2550 50  0001 C CNN
+F 3 "" H 6050 2550 50  0001 C CNN
+	1    6050 2550
+	1    0    0    -1
+$EndComp
+Wire Wire Line
+	5900 2200 6050 2200
+Wire Wire Line
+	6050 2200 6050 2250
+Wire Wire Line
+	6050 2200 6200 2200
+Connection ~ 6050 2200
 $EndSCHEMATC

Commit message: More c++ code, bug fixes on the PCB
Parts:
- R4: value 5k / 47k ? -> 6k8
- gave numbers to parts that had none: 2
Changed lines of the file:
@@
 P 4100 1700
 F 0 "R4" V 3893 1700 50  0000 C CNN
-F 1 "5k / 47k ?" V 3984 1700 50  0000 C CNN
+F 1 "6k8" V 3984 1700 50  0000 C CNN
 F 2 "Resistors_SMD:R_0805" V 4030 1700 50  0001 C CNN
 F 3 "~" H 4100 1700 50  0001 C CNN
@@
 	2950 1650 4700 1650
 $Comp
-L Device:R R?
+L Device:R R24
 U 1 1 5B9E9754
 P 5750 2200
-F 0 "R?" V 5543 2200 50  0000 C CNN
+F 0 "R24" V 5543 2200 50  0000 C CNN
 F 1 "1k1" V 5634 2200 50  0000 C CNN
 F 2 "Resistors_SMD:R_0805" V 5680 2200 50  0001 C CNN
@@
 $EndComp
 $Comp
-L Device:CP C?
+L Device:CP C21
 U 1 1 5B9E9EC7
 P 6050 2400
-F 0 "C?" H 6168 2446 50  0000 L CNN
+F 0 "C21" H 6168 2446 50  0000 L CNN
 F 1 "10u" H 6168 2355 50  0000 L CNN
 F 2 "Capacitors_SMD:CP_Elec_4x5.8" H 6088 2250 50  0001 C CNN
@@
 NoConn ~ 5450 2800
 $Comp
-L power:GND #PWR?
+L power:GND #PWR0132
 U 1 1 5BA11FCB
 P 6050 2550
-F 0 "#PWR?" H 6050 2300 50  0001 C CNN
+F 0 "#PWR0132" H 6050 2300 50  0001 C CNN
 F 1 "GND" H 6055 2377 50  0000 C CNN
 F 2 "" H 6050 2550 50  0001 C CNN

Commit message: BCB fixes and cpp code mostly done
Parts:
- Q1: value STP60NF06L -> STP60NF06L / STP9NK60Z
- R15, R19: value 5k -> 15k
- U2: value LM78M12 -> LM78M09
Changed lines of the file:
@@
 P 5350 1800
 F 0 "Q1" H 5555 1846 50  0000 L CNN
-F 1 "STP60NF06L" H 5555 1755 50  0000 L CNN
+F 1 "STP60NF06L / STP9NK60Z" H 5555 1755 50  0000 L CNN
 F 2 "TO_SOT_Packages_THT:TO-220-3_Vertical" H 5550 1900 50  0001 C CNN
 F 3 "~" H 5350 1800 50  0001 C CNN
@@
 P 1550 3200
 F 0 "U2" H 1550 3442 50  0000 C CNN
-F 1 "LM78M12" H 1550 3351 50  0000 C CNN
+F 1 "LM78M09" H 1550 3351 50  0000 C CNN
 F 2 "TO_SOT_Packages_SMD:TO-252-2_Rectifier" H 1550 3425 50  0001 C CIN
 F 3 "http://www.fairchildsemi.com/ds/LM/LM7805.pdf" H 1550 3150 50  0001 C CNN
@@
 P 6300 6150
 F 0 "R15" H 6230 6104 50  0000 R CNN
-F 1 "5k" H 6230 6195 50  0000 R CNN
+F 1 "15k" H 6230 6195 50  0000 R CNN
 F 2 "Resistors_SMD:R_0805" V 6230 6150 50  0001 C CNN
 F 3 "~" H 6300 6150 50  0001 C CNN
@@
 P 8900 6150
 F 0 "R19" H 8830 6104 50  0000 R CNN
-F 1 "5k" H 8830 6195 50  0000 R CNN
+F 1 "15k" H 8830 6195 50  0000 R CNN
 F 2 "Resistors_SMD:R_0805" V 8830 6150 50  0001 C CNN
 F 3 "~" H 8900 6150 50  0001 C CNN

Commit message: major schematic work
Parts:
- U3: symbol MCU_Microchip_ATmega:ATxmega32E5-AU -> ActiveLoadMosfets-rescue:ATxmega32E5-AU-MCU_Microchip_ATmega
- U4, U8: symbol myLib:LED-3digits -> ActiveLoadMosfets-rescue:LED-3digits-myLib
- U6, U7: symbol myLib:SCT2167 -> ActiveLoadMosfets-rescue:SCT2167-myLib
Changed lines of the file:
@@
 $EndComp
 $Comp
-L myLib:LED-3digits U4
+L ActiveLoadMosfets-rescue:LED-3digits-myLib U4
 U 1 1 5B775CCD
 P 10700 4750
@@
 $EndComp
 $Comp
-L MCU_Microchip_ATmega:ATxmega32E5-AU U3
+L ActiveLoadMosfets-rescue:ATxmega32E5-AU-MCU_Microchip_ATmega U3
 U 1 1 5B775F7C
 P 3450 6100
@@
 $EndComp
 $Comp
-L myLib:SCT2167 U6
+L ActiveLoadMosfets-rescue:SCT2167-myLib U6
 U 1 1 5B7BA647
 P 9650 5800
@@
 	8100 2600 8100 2700
 $Comp
-L myLib:LED-3digits U8
+L ActiveLoadMosfets-rescue:LED-3digits-myLib U8
 U 1 1 5BB37628
 P 8100 4750
@@
 $EndComp
 $Comp
-L myLib:SCT2167 U7
+L ActiveLoadMosfets-rescue:SCT2167-myLib U7
 U 1 1 5BB3762E
 P 7050 5800
