File: KiCad/ActiveLoadMosfets/ActiveLoadMosfets.kicad_pcb (KiCad board)
At the start: 2 copper layers, 30 parts, among them J1 Conn_01x02_Male, Q1 STP60NF06L, Q2 STP60NF06L, Q3 STP60NF06L, Q4 STP60NF06L, Q5 STP60NF06L, Q6 STP60NF06L, U1 LM7322, U2 LM78M12

Commit message: pcb work
Parts:
- added C10: 10u, Capacitors_SMD:CP_Elec_4x5.8, F.Cu at (106.0, 64.8)
- added C11: 100n, Capacitors_SMD:C_0805, F.Cu at (111.5, 66.0)
- added C12: 10u, Capacitors_SMD:CP_Elec_4x5.8, F.Cu at (106.0, 45.1)
- added C13: 100n, Capacitors_SMD:C_0805, F.Cu at (100.3, 45.7)
- added C14: 10n, Capacitors_SMD:C_0805, F.Cu at (85.1, 76.8)
- added C15: 100n, Capacitors_SMD:C_0805, F.Cu at (110.5, 149.2)
- added C16: 100n, Capacitors_SMD:C_0805, F.Cu at (134.4, 143.1)
- added C17: 1u, Capacitors_SMD:C_0805, F.Cu at (85.1, 80.0)
- added C18: 1u, Capacitors_SMD:C_0805, F.Cu at (136.5, 71.8)
- added C19: 10n, Capacitors_SMD:C_0805, F.Cu at (137.2, 74.3)
- added C7: 47u, Capacitors_SMD:CP_Elec_6.3x5.8, F.Cu at (83.8, 126.4)
- added C8: 100n, Capacitors_SMD:C_0805, F.Cu at (106.7, 86.4)
- added C9: 47u, Capacitors_SMD:CP_Elec_6.3x5.8, F.Cu at (108.0, 76.8)
- added J2: Conn_02x03_Odd_Even, Pin_Headers:Pin_Header_Straight_2x03_Pitch2.54mm, F.Cu at (105.4, 32.4)
- added L1: 10u, Inductors_SMD:L_0805, F.Cu at (112.4, 62.2)
- added Q7: IRLML2244, TO_SOT_Packages_SMD:SOT-23, F.Cu at (82.5, 40.0)
- added Q8: IRLML2244, TO_SOT_Packages_SMD:SOT-23, F.Cu at (113.0, 38.1)
- added Q9: IRLML2244, TO_SOT_Packages_SMD:SOT-23, F.Cu at (130.2, 40.0)
- added R14: 10k, Resistors_SMD:R_0805, F.Cu at (96.2, 67.9)
- added R15: 1k, Resistors_SMD:R_0805, F.Cu at (135.3, 81.9)
- added R16: 1k, Resistors_SMD:R_0805, F.Cu at (70.5, 73.7)
- added R17: 1k, Resistors_SMD:R_0805, F.Cu at (70.5, 77.5)
- added R18: 10, Resistors_SMD:R_1206, F.Cu at (134.6, 85.7)
- added R19: 1k, Resistors_SMD:R_0805, F.Cu at (77.5, 85.7)
- added R20: 10, Resistors_SMD:R_1206, F.Cu at (81.9, 87.0)
- added REF**: MountingHole_6mm, Mounting_Holes:MountingHole_6mm, F.Cu at (104.1, 121.9)
- added REF**: MountingHole_6mm, Mounting_Holes:MountingHole_6mm, F.Cu at (134.6, 121.3)
- added REF**: MountingHole_3.2mm_M3, Mounting_Holes:MountingHole_3.2mm_M3, F.Cu at (67.9, 169.5)
- added REF**: MountingHole_3.2mm_M3, Mounting_Holes:MountingHole_3.2mm_M3, F.Cu at (146.1, 168.3)
- added REF**: MountingHole_3.2mm_M3, Mounting_Holes:MountingHole_3.2mm_M3, F.Cu at (146.7, 19.7)
- added REF**: MountingHole_3.2mm_M3, Mounting_Holes:MountingHole_3.2mm_M3, F.Cu at (68.6, 19.1)
- added U3: ATxmega32E5-AU, Housings_QFP:TQFP-32_7x7mm_Pitch0.8mm, F.Cu at (105.4, 55.9)
- added U4: LED-3digits, JPDisplays:LED-14.2x3, F.Cu at (128.3, 55.9)
- added U5: LM78M33, TO_SOT_Packages_SMD:TO-252-2_Rectifier, F.Cu at (97.2, 84.7)
- added U6: SCT2167, Housings_SOIC:SOIC-16_3.9x9.9mm_Pitch1.27mm, F.Cu at (125.1, 55.2)
- added U7: SCT2167, Housings_SOIC:SOIC-16_3.9x9.9mm_Pitch1.27mm, F.Cu at (87.6, 56.5)
- added U8: LED-3digits, JPDisplays:LED-14.2x3, F.Cu at (83.8, 55.9)
- C6: value 10u -> 47u; footprint Capacitors_SMD:CP_Elec_4x5.8 -> Capacitors_SMD:CP_Elec_6.3x5.8
- R6: moved to B.Cu
- RV1, RV2: footprint Pin_Headers:Pin_Header_Straight_1x03_Pitch2.54mm -> Connectors_Terminal_Blocks:TerminalBlock_bornier-3_P5.08mm
- moved R8 117.6 mm to (132.1, 156.8), turned to 180 degrees
- moved R12 97.9 mm to (135.3, 31.1)
- moved R7 91.9 mm to (80.0, 31.8), turned to 90 degrees
- moved RV1 87.8 mm to (99.1, 135.9)
- moved J1 77.1 mm to (72.4, 123.8), turned to 270 degrees
- moved U1 76.6 mm to (120.0, 95.9)
- moved Q2 73.7 mm to (140.8, 155.6)
- moved C5 58.9 mm to (121.9, 92.1), turned to 180 degrees
- moved C3 58.1 mm to (118.1, 99.7)
- moved Q4 56.5 mm to (71.9, 160.7)
- moved Q5 56.5 mm to (140.8, 29.2)
- moved R9 55.1 mm to (138.1, 148.0)
- moved R13 52.5 mm to (139.4, 85.1)
- moved C6 48.4 mm to (99.7, 103.5)
- moved C1 47.7 mm to (118.1, 101.6), turned to 180 degrees
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Connections:
- net Net-(Q1-Pad3) renamed CURRENT
- RV2 pad 1: (no net) -> Net-(RV2-Pad1)
Routing:
- net CURRENT: track 0.00 -> 364.2 mm
- net VDD: track 0.00 -> 283.9 mm
- net GND: track 0.00 -> 39.2 mm
- net Net-(R3-Pad2): track 0.00 -> 15.7 mm
- net Net-(C5-Pad2): track 0.00 -> 9.48 mm
- net Net-(R6-Pad2): track 0.00 -> 9.37 mm, vias 0 -> 1
- net +12V: track 0.00 -> 8.05 mm
- net Net-(C1-Pad1): track 0.00 -> 6.63 mm
- net Net-(C5-Pad1): track 0.00 -> 5.94 mm
- net Net-(R3-Pad1): track 0.00 -> 5.25 mm
Other:
- board outline added: 90.8 x 161.9 mm
- net class Default: trace_width 0.25 -> 0.5588; via_dia 0.8 -> 1.4; via_drill 0.4 -> 0.6
- net class Power added: clearance 0.2, trace_width 2, via_dia 2, via_drill 0.8

Commit message: More pcb work
Parts:
- removed REF** (x2): MountingHole_6mm, Mounting_Holes:MountingHole_6mm
- removed REF** (x4): MountingHole_3.2mm_M3, Mounting_Holes:MountingHole_3.2mm_M3
- added C20: 10n, Capacitors_SMD:C_0805, F.Cu at (118.7, 36.5)
- added D1: LED, LEDs:LED_0805, F.Cu at (88.9, 35.2)
- added R21: 10k, Resistors_SMD:R_0805, F.Cu at (92.1, 35.2)
- added R22: 10k, Resistors_SMD:R_0805, F.Cu at (116.8, 36.2)
- added R23: 10k, Resistors_SMD:R_0805, F.Cu at (116.8, 32.1)
- added SW1: SW_SPST, Buttons_Switches_SMD:SW_SPST_B3SL-1002P, F.Cu at (124.5, 34.0)
- C10: value 10u -> 100n; footprint Capacitors_SMD:CP_Elec_4x5.8 -> Capacitors_SMD:C_0805
- moved C15 79.2 mm to (118.7, 70.4), turned to 270 degrees
- moved C16 74.4 mm to (122.8, 69.5), turned to 180 degrees
- moved R16 55.3 mm to (125.7, 71.4)
- moved R17 52.7 mm to (122.9, 71.4)
- moved R19 52.0 mm to (120.0, 55.9), turned to 90 degrees
- moved R20 51.2 mm to (118.1, 50.8), turned to 90 degrees
- moved R15 50.4 mm to (92.1, 55.9), turned to 270 degrees
- moved R18 47.6 mm to (94.0, 61.0), turned to 270 degrees
- moved R14 33.5 mm to (99.1, 34.6), turned to 90 degrees
- moved Q8 28.1 mm to (85.1, 40.6), turned to 270 degrees
- moved C19 27.9 mm to (116.2, 55.9), turned to 90 degrees
- moved C17 26.4 mm to (95.9, 55.9), turned to 270 degrees
- moved C18 24.3 mm to (118.1, 55.9), turned to 90 degrees
- moved C14 22.8 mm to (94.0, 55.9), turned to 270 degrees
- moved C4 19.8 mm to (89.2, 92.1), turned to 180 degrees
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Connections:
- net Net-(C12-Pad1) renamed /+3.3Va
- C11 pad 1: +3V3 -> GND
- C11 pad 2: GND -> +3V3
- C8 pad 1: +3V3 -> +12V
- U3 pad 24: Net-(U3-Pad24) -> CURRENT
- U3 pad 25: Net-(U3-Pad25) -> VOLTAGE
- U3 pad 4: CURRENT -> Net-(U3-Pad4)
- U3 pad 5: VOLTAGE -> Net-(U3-Pad5)
- U6 pad 10: Net-(U4-Pad10) -> Net-(U4-Pad5)
- U6 pad 11: Net-(U4-Pad5) -> Net-(U4-Pad10)
- U6 pad 12: Net-(U4-Pad3) -> Net-(U4-Pad11)
- U6 pad 15: Net-(R15-Pad2) -> Net-(R19-Pad2)
- U6 pad 16: Net-(C14-Pad2) -> Net-(C18-Pad2)
- U6 pad 2: MOSI -> Net-(U6-Pad2)
- U6 pad 5: Net-(U4-Pad11) -> Net-(U4-Pad1)
- U6 pad 6: Net-(U4-Pad7) -> Net-(U4-Pad2)
- U6 pad 7: Net-(U4-Pad4) -> Net-(U4-Pad3)
- U6 pad 8: Net-(U4-Pad2) -> Net-(U4-Pad4)
- U6 pad 9: Net-(U4-Pad1) -> Net-(U4-Pad7)
- U7 pad 13: Net-(U7-Pad13) -> OutputEnabled
- U7 pad 14: Net-(U7-Pad14) -> Net-(U6-Pad2)
- U7 pad 15: Net-(R19-Pad2) -> Net-(R15-Pad2)
- U7 pad 16: Net-(C18-Pad2) -> Net-(C14-Pad2)
- U7 pad 2: Net-(U6-Pad14) -> MOSI
- U8 pad 1: Net-(U7-Pad9) -> Net-(U7-Pad7)
- U8 pad 10: Net-(U7-Pad10) -> Net-(U7-Pad6)
- U8 pad 11: Net-(U7-Pad5) -> Net-(U7-Pad8)
- U8 pad 2: Net-(U7-Pad8) -> Net-(U7-Pad9)
- U8 pad 3: Net-(U7-Pad12) -> Net-(U7-Pad10)
- U8 pad 4: Net-(U7-Pad7) -> Net-(U7-Pad11)
- U8 pad 5: Net-(U7-Pad11) -> Net-(U7-Pad12)
- U8 pad 7: Net-(U7-Pad6) -> Net-(U7-Pad5)
Routing:
- net Net-(C5-Pad1): track 5.94 -> 318.8 mm, vias 0 -> 3
- net GND: track 39.2 -> 284.5 mm, vias 0 -> 8
- net +3V3: track 0.00 -> 123.7 mm, vias 0 -> 2
- net VDD: track 283.9 -> 357.7 mm, vias 0 -> 1
- net +12V: track 8.05 -> 75.6 mm
- net OutputEnabled: track 0.00 -> 56.1 mm, vias 0 -> 3
- net Net-(Q9-Pad3): track 0.00 -> 55.1 mm, vias 0 -> 2
- net Net-(Q8-Pad3): track 0.00 -> 54.5 mm, vias 0 -> 2
- net Net-(Q7-Pad3): track 0.00 -> 53.6 mm, vias 0 -> 2
- net Latch: track 0.00 -> 50.5 mm, vias 0 -> 3
- net CURRENT: track 364.2 -> 410.7 mm, vias 0 -> 1
- net SCK: track 0.00 -> 46.3 mm, vias 0 -> 3
- net Digit1: track 0.00 -> 44.1 mm, vias 0 -> 2
- net Digit2: track 0.00 -> 40.8 mm, vias 0 -> 2
- net Net-(R2-Pad2): track 0.00 -> 40.3 mm
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Other:
- board size 90.8 x 161.9 mm -> 83.2 x 161.9 mm
- net class SmallPower added: clearance 0.2, trace_width 1.016, via_dia 1.4, via_drill 0.6

Commit message: PCB Proofed
Parts:
- added REF**: MountingHole_3.2mm_M3, Mounting_Holes:MountingHole_3.2mm_M3, F.Cu at (70.5, 19.7)
- added REF**: MountingHole_3.2mm_M3, Mounting_Holes:MountingHole_3.2mm_M3, F.Cu at (141.6, 19.7)
- added REF**: MountingHole_3.2mm_M3, Mounting_Holes:MountingHole_3.2mm_M3, F.Cu at (141.6, 169.5)
- added REF**: MountingHole_3.2mm_M3, Mounting_Holes:MountingHole_3.2mm_M3, F.Cu at (70.5, 169.5)
- added REF**: MountingHole_3.2mm_M3, Mounting_Holes:MountingHole_3.2mm_M3, F.Cu at (76.2, 76.2)
- added REF**: MountingHole_3.2mm_M3, Mounting_Holes:MountingHole_3.2mm_M3, F.Cu at (136.5, 108.0)
- added SW2: SW_SPDT, JPConnectors:SlideSwitch3Poles, F.Cu at (89.5, 76.2)
- RV1, RV2: footprint Connectors_Terminal_Blocks:TerminalBlock_bornier-3_P5.08mm -> JPResistors:Pot_PCB-mount
- SW1: footprint Buttons_Switches_SMD:SW_SPST_B3SL-1002P -> Buttons_Switches_SMD:SW_SPST_B3S-1000
- moved R1 31.2 mm to (111.1, 104.1)
- moved C7 19.7 mm to (87.6, 107.0), turned to 180 degrees
- moved RV2 6.35 mm to (134.6, 139.7), turned to 0 degrees
- moved RV1 4.26 mm to (101.0, 139.7)
- moved C12 3.18 mm to (108.0, 43.2)
- moved C10 2.54 mm to (104.1, 76.2)
- moved C8 2.54 mm to (104.1, 86.4)
- moved U5 2.54 mm to (102.2, 81.3)
- moved C9 2.54 mm to (106.0, 71.8)
- moved SW1 1.91 mm to (126.4, 34.0)
- moved R6 1.71 mm to (129.2, 97.2)
- moved C20 0.95 mm to (118.7, 35.6)
- moved R14 0.95 mm to (99.1, 33.7)
- moved R22 0.64 mm to (116.8, 35.6)
Connections:
- C8 pad 1: +12V -> Net-(C8-Pad1)
- J2 pad 3: Net-(J2-Pad3) -> (no net)
- J2 pad 4: Net-(J2-Pad4) -> (no net)
- RV1 pad 1: Net-(R1-Pad1) -> Net-(RV1-Pad1)
- RV1 pad 3: Net-(RV1-Pad3) -> Net-(R1-Pad1)
- RV2 pad 1: Net-(RV2-Pad1) -> GND
- RV2 pad 2: Net-(RV1-Pad3) -> Net-(RV1-Pad1)
- RV2 pad 3: GND -> (no net)
- U3 pad 10: Net-(U3-Pad10) -> (no net)
- U3 pad 12: Net-(U3-Pad12) -> (no net)
- U3 pad 13: Net-(U3-Pad13) -> SWITCH
- U3 pad 14: Net-(U3-Pad14) -> LED
- U3 pad 19: Net-(U3-Pad19) -> (no net)
- U3 pad 2: Net-(U3-Pad2) -> (no net)
- U3 pad 20: Net-(U3-Pad20) -> (no net)
- U3 pad 21: Net-(U3-Pad21) -> (no net)
- U3 pad 22: Net-(U3-Pad22) -> (no net)
- U3 pad 23: Net-(U3-Pad23) -> (no net)
- U3 pad 26: Net-(U3-Pad26) -> (no net)
- U3 pad 27: Net-(U3-Pad27) -> (no net)
- U3 pad 28: Net-(U3-Pad28) -> (no net)
- U3 pad 3: Net-(U3-Pad3) -> (no net)
- U3 pad 4: Net-(U3-Pad4) -> (no net)
- U3 pad 5: Net-(U3-Pad5) -> (no net)
- U3 pad 6: Net-(U3-Pad6) -> (no net)
- U5 pad 1: +12V -> Net-(C8-Pad1)
- U6 pad 14: Net-(U6-Pad14) -> (no net)
Routing:
- net GND: track 284.5 -> 372.1 mm, vias 8 -> 9
- net +3V3: track 123.7 -> 187.5 mm, vias 2 -> 3
- net VDD: track 357.7 -> 416.8 mm, vias 1 -> 2
- net Net-(RV1-Pad1): track 0.00 -> 46.4 mm
- net SWITCH: track 2.06 -> 42.0 mm, vias 0 -> 2
- net Net-(R1-Pad1): track 8.36 -> 40.2 mm, vias 0 -> 1
- net Net-(RV1-Pad3): track 28.8 -> 0.00 mm
- net LED: track 0.00 -> 26.8 mm
- net Net-(C8-Pad1): track 0.00 -> 24.9 mm, vias 0 -> 1
- net Net-(R2-Pad2): track 40.3 -> 58.1 mm, vias 0 -> 1
- net Net-(C5-Pad1): track 318.8 -> 331.7 mm
- net +12V: track 75.6 -> 66.8 mm, vias 0 -> 2
- net (no net): track 0.00 -> 4.45 mm
- net Net-(R22-Pad1): track 13.2 -> 15.6 mm
- net /+3.3Va: track 10.6 -> 12.8 mm
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- added copper zone on F.Cu, net GND
Other:
- board text added: "0.1R / 10W"
- board text added: "ActiveLoadMosfets v1 JP, 20.08.2018"
- board text added: "Gnd 13.8-35V"
- board text added: "Vdd"

Commit message: PCB proofing
Parts:
- moved REF** 6.38 mm to (74.0, 82.2)
- moved REF** 2.59 mm to (139.0, 107.2)
Other:
- board text added: "ActiveLoadMosfets v1 JP, 21.08.2018"
- board text removed: "ActiveLoadMosfets v1 JP, 20.08.2018"
Changed lines of the file:
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@@
     (mod_text_size 1 1)
     (mod_text_width 0.15)
-    (pad_size 2.7 2.7)
-    (pad_drill 2.7)
+    (pad_size 3.2 3.2)
+    (pad_drill 3.2)
     (pad_to_mask_clearance 0.2)
     (aux_axis_origin 0 0)
@@
     (fp_circle (center 0 0) (end 3.2 0) (layer Cmts.User) (width 0.15))
     (fp_circle (center 0 0) (end 3.45 0) (layer F.CrtYd) (width 0.05))
-    (pad 1 np_thru_hole circle (at 0 0) (size 3.2 3.2) (drill 3.2) (layers *.Cu *.Mask))
+    (pad "" np_thru_hole circle (at 0 0) (size 3.2 3.2) (drill 3.2) (layers *.Cu *.Mask)
+      (clearance 3.25))
   )
   (module Mounting_Holes:MountingHole_3.2mm_M3 (layer F.Cu)
-    (at 76.2 76.2)
+    (at 74 82.185)
     (descr "Mounting Hole 3.2mm, no annular, M3")
     (tags "mounting hole 3.2mm no annular m3")
@@
     (fp_circle (center 0 0) (end 3.2 0) (layer Cmts.User) (width 0.15))
     (fp_circle (center 0 0) (end 3.45 0) (layer F.CrtYd) (width 0.05))
-    (pad 1 np_thru_hole circle (at 0 0) (size 3.2 3.2) (drill 3.2) (layers *.Cu *.Mask))
+    (pad "" np_thru_hole circle (at 0 0) (size 3.2 3.2) (drill 3.2) (layers *.Cu *.Mask)
+      (clearance 3.25))
   )
   (module Mounting_Holes:MountingHole_3.2mm_M3 (layer F.Cu)
-    (at 136.525 107.95)
+    (at 139 107.185)
     (descr "Mounting Hole 3.2mm, no annular, M3")
     (tags "mounting hole 3.2mm no annular m3")
@@
     (effects (font (size 2.54 2.54) (thickness 0.508)) (justify mirror))
   )
-  (gr_text "ActiveLoadMosfets v1\nJP, 20.08.2018" (at 106.045 20.32) (layer F.Cu)
+  (gr_text "ActiveLoadMosfets v1\nJP, 21.08.2018" (at 106.045 20.32) (layer F.Cu)
     (effects (font (size 2.54 2.54) (thickness 0.508)))
   )
@@
   (segment (start 84.455 108.585) (end 84.455 104.14) (width 1.016) (layer B.Cu) (net 2))
   (segment (start 84.455 104.14) (end 84.455 102.235) (width 1.016) (layer B.Cu) (net 2))
-  (segment (start 116.84 104.14) (end 120.65 104.14) (width 1.016) (layer B.Cu) (net 2))
-  (segment (start 120.65 104.14) (end 123.825 107.315) (width 1.016) (layer B.Cu) (net 2))
-  (segment (start 126.365 139.7) (end 129.62 139.7) (width 1.016) (layer B.Cu) (net 2))
-  (segment (start 123.825 107.315) (end 123.825 137.16) (width 1.016) (layer B.Cu) (net 2))
-  (segment (start 123.825 137.16) (end 126.365 139.7) (width 1.016) (layer B.Cu) (net 2))
   (segment (start 106.95 48.895) (end 106.95 46.625) (width 1.016) (layer F.Cu) (net 2))
   (segment (start 106.15 45.825) (end 106.15 43.18) (width 1.016) (layer F.Cu) (net 2))
@@
   (segment (start 122.39 36.225) (end 124.46 36.225) (width 1.016) (layer F.Cu) (net 2))
   (segment (start 124.46 36.225) (end 130.34 36.225) (width 1.016) (layer F.Cu) (net 2))
+  (segment (start 126.365 139.7) (end 129.62 139.7) (width 1.016) (layer B.Cu) (net 2))
+  (segment (start 123.19 136.525) (end 126.365 139.7) (width 1.016) (layer B.Cu) (net 2))
+  (segment (start 123.19 106.68) (end 123.19 136.525) (width 1.016) (layer B.Cu) (net 2))
+  (segment (start 116.84 104.14) (end 120.65 104.14) (width 1.016) (layer B.Cu) (net 2))
+  (segment (start 120.65 104.14) (end 123.19 106.68) (width 1.016) (layer B.Cu) (net 2))
   (segment (start 71.905 31.75) (end 69.85 31.75) (width 2) (layer F.Cu) (net 3))
   (segment (start 69.85 31.75) (end 66.675 34.925) (width 2) (layer F.Cu) (net 3))
@@
   (segment (start 92.205 94.875) (end 92.205 92.075) (width 1.016) (layer F.Cu) (net 4))
   (segment (start 92.205 92.075) (end 92.205 87.66) (width 1.016) (layer F.Cu) (net 4))
-  (segment (start 105.14 86.36) (end 106.045 86.36) (width 1.016) (layer F.Cu) (net 60))
-  (segment (start 106.045 86.36) (end 106.68 85.725) (width 1.016) (layer F.Cu) (net 60))
-  (segment (start 106.81 85.596) (end 106.81 83.58) (width 1.016) (layer F.Cu) (net 60))
-  (segment (start 106.681 85.725) (end 106.81 85.596) (width 1.016) (layer F.Cu) (net 60))
-  (segment (start 106.68 85.725) (end 106.681 85.725) (width 1.016) (layer F.Cu) (net 60))
   (segment (start 111.125 99.38) (end 120.65 99.38) (width 1.016) (layer B.Cu) (net 4))
   (segment (start 120.335 99.695) (end 120.65 99.38) (width 1.016) (layer F.Cu) (net 4))
@@
   (segment (start 125.095 92.075) (end 134.6662 92.075) (width 1.016) (layer F.Cu) (net 6))
   (via (at 90.17 109.855) (size 1.4) (drill 0.6) (layers F.Cu B.Cu) (net 6))
-  (segment (start 134.62 100.965) (end 134.62 91.76) (width 1.016) (layer F.Cu) (net 6))
-  (via (at 121.285 108.585) (size 1.4) (drill 0.6) (layers F.Cu B.Cu) (net 6))
   (segment (start 76.2 104.14) (end 72.39 104.14) (width 1.016) (layer F.Cu) (net 6))
   (segment (start 81.915 109.855) (end 76.2 104.14) (width 1.016) (layer F.Cu) (net 6))
   (segment (start 90.17 109.855) (end 81.915 109.855) (width 1.016) (layer F.Cu) (net 6))
-  (segment (start 121.285 108.585) (end 127 108.585) (width 1.016) (layer F.Cu) (net 6))
-  (segment (start 127 108.585) (end 134.62 100.965) (width 1.016) (layer F.Cu) (net 6))
   (via (at 120.015 142.24) (size 1.4) (drill 0.6) (layers F.Cu B.Cu) (net 6))
-  (segment (start 121.285 108.585) (end 120.015 108.585) (width 1.016) (layer B.Cu) (net 6))
   (segment (start 136.21 153.035) (end 120.015 153.035) (width 1.016) (layer F.Cu) (net 6))
   (segment (start 112.395 160.655) (end 77.15 160.655) (width 1.016) (layer F.Cu) (net 6))
@@
   (segment (start 120.015 142.24) (end 120.015 153.035) (width 1.016) (layer F.Cu) (net 6))
   (segment (start 120.015 108.585) (end 120.015 142.24) (width 1.016) (layer B.Cu) (net 6))
+  (via (at 120.65 108.585) (size 1.4) (drill 0.6) (layers F.Cu B.Cu) (net 6))
+  (segment (start 120.65 108.585) (end 120.015 108.585) (width 1.016) (layer B.Cu) (net 6))
+  (segment (start 134.62 100.965) (end 134.62 91.76) (width 1.016) (layer F.Cu) (net 6))
+  (segment (start 127 108.585) (end 134.62 100.965) (width 1.016) (layer F.Cu) (net 6))
+  (segment (start 120.65 108.585) (end 127 108.585) (width 1.016) (layer F.Cu) (net 6))
   (segment (start 71.905 34.29) (end 75.25 34.29) (width 1.016) (layer F.Cu) (net 7))
   (segment (start 140.65 155.575) (end 138.11 153.035) (width 1.016) (layer F.Cu) (net 8))
@@
   (segment (start 111.125 107.95) (end 111.125 105.09) (width 1.016) (layer F.Cu) (net 13))
   (segment (start 113.03 109.855) (end 111.125 107.95) (width 1.016) (layer F.Cu) (net 13))
-  (segment (start 109.14 139.7) (end 105.965 139.7) (width 1.016) (layer B.Cu) (net 13))
-  (segment (start 113.03 109.855) (end 113.03 135.81) (width 1.016) (layer B.Cu) (net 13))
-  (segment (start 113.03 135.81) (end 109.14 139.7) (width 1.016) (layer B.Cu) (net 13))
+  (segment (start 109.855 139.7) (end 105.965 139.7) (width 1.016) (layer B.Cu) (net 13))
+  (segment (start 113.03 109.855) (end 113.03 136.525) (width 1.016) (layer B.Cu) (net 13))
+  (segment (start 113.03 136.525) (end 109.855 139.7) (width 1.016) (layer B.Cu) (net 13))
   (segment (start 122.555 103.505) (end 122.555 102.87) (width 1.016) (layer F.Cu) (net 14))
   (segment (start 116.205 109.855) (end 122.555 103.505) (width 1.016) (layer F.Cu) (net 14))
@@
   (segment (start 100.965 141.605) (end 100.965 139.7) (width 1.016) (layer B.Cu) (net 14))
   (segment (start 102.235 142.875) (end 100.965 141.605) (width 1.016) (layer B.Cu) (net 14))
-  (segment (start 112.395 142.875) (end 102.235 142.875) (width 1.016) (layer B.Cu) (net 14))
-  (segment (start 116.205 109.855) (end 116.205 139.065) (width 1.016) (layer B.Cu) (net 14))
-  (segment (start 116.205 139.065) (end 112.395 142.875) (width 1.016) (layer B.Cu) (net 14))
+  (segment (start 111.76 142.875) (end 102.235 142.875) (width 1.016) (layer B.Cu) (net 14))
+  (segment (start 116.205 109.855) (end 116.205 138.43) (width 1.016) (layer B.Cu) (net 14))
+  (segment (start 116.205 138.43) (end 111.76 142.875) (width 1.016) (layer B.Cu) (net 14))
   (segment (start 115.5088 93.345) (end 116.1438 93.98) (width 0.5588) (layer F.Cu) (net 15))
   (segment (start 114.3 93.345) (end 115.5088 93.345) (width 0.5588) (layer F.Cu) (net 15))
@@
   (segment (start 95.965 139.7) (end 95.965 142.32) (width 1.016) (layer B.Cu) (net 59))
   (segment (start 95.965 142.32) (end 99.06 145.415) (width 1.016) (layer B.Cu) (net 59))
+  (segment (start 105.14 86.36) (end 106.045 86.36) (width 1.016) (layer F.Cu) (net 60))
+  (segment (start 106.045 86.36) (end 106.68 85.725) (width 1.016) (layer F.Cu) (net 60))
+  (segment (start 106.81 85.596) (end 106.81 83.58) (width 1.016) (layer F.Cu) (net 60))
+  (segment (start 106.681 85.725) (end 106.81 85.596) (width 1.016) (layer F.Cu) (net 60))
+  (segment (start 106.68 85.725) (end 106.681 85.725) (width 1.016) (layer F.Cu) (net 60))
   (via (at 107.315 86.36) (size 1.4) (drill 0.6) (layers F.Cu B.Cu) (net 60))
   (segment (start 104.395 83.44) (end 107.315 86.36) (width 1.016) (layer B.Cu) (net 60))
